File: kicad/ESP32-wood-beam-lamp.sch (KiCad schematic (older format))
At the start: 48 parts, among them J1 Screw_Terminal_01x05, J2 Screw_Terminal_01x05, J3 Serial-Prog, J4 Conn_01x02, J5 NextionDisplay, J6 USB_B_Micro, J7 AUX, Q1 IRF3708, Q2 IRF3708, SW1 Flash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

Commit message: footprints added
Parts:
- J3, J7: footprint Connector_PinHeader_2.54mm:PinHeader_1x05_P2.54mm_Horizontal -> Connector_PinHeader_2.54mm:PinHeader_1x05_P2.54mm_Vertical
Connections:
- no-connect marks 31 -> 32
Changed lines of the file:
@@
 F 0 "J3" H 3950 3500 50  0000 R CNN
 F 1 "Serial-Prog" H 4150 3600 50  0000 R CNN
-F 2 "Connector_PinHeader_2.54mm:PinHeader_1x05_P2.54mm_Horizontal" H 3950 3200 50  0001 C CNN
+F 2 "Connector_PinHeader_2.54mm:PinHeader_1x05_P2.54mm_Vertical" H 3950 3200 50  0001 C CNN
 F 3 "~" H 3950 3200 50  0001 C CNN
 	1    3950 3200
@@
 F 0 "J7" H 1150 5600 50  0000 R CNN
 F 1 "AUX" H 1150 5700 50  0000 R CNN
-F 2 "Connector_PinHeader_2.54mm:PinHeader_1x05_P2.54mm_Horizontal" H 1150 5300 50  0001 C CNN
+F 2 "Connector_PinHeader_2.54mm:PinHeader_1x05_P2.54mm_Vertical" H 1150 5300 50  0001 C CNN
 F 3 "~" H 1150 5300 50  0001 C CNN
 	1    1150 5300
@@
 NoConn ~ 9100 4200
 NoConn ~ 9100 4300
+NoConn ~ 150  3200
 $EndSCHEMATC

Commit message: rotary Encoder added
Parts:
- added C7, C9: 1u, symbol Device:C
- added R11, R9: 10K, symbol Device:R
- added SW3: Rotary_Encoder_Switch, symbol Device:Rotary_Encoder_Switch
Connections:
- net +3V3: now also R11.1, R9.1
- net GND: now also C7.2, C9.2, SW3.C, SW3.S2
- net ROT_A: now reaches U2.12 (IO27)
- net ROT_A: now also C7.1, R9.2, SW3.A
- net ROT_B: now reaches U2.13 (IO14)
- net ROT_B: now also C9.1, R11.2, SW3.B
- net ROT_SW: now reaches U2.14 (IO12)
- net ROT_SW: now also SW3.S1
- no-connect marks 32 -> 29
Other:
- moved on the sheet: C1, C3, C4, D4, D5, J3, J7, Q1, Q2, R1, R13, R2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
