File: kicad/ESP32-wood-beam-lamp.sch (KiCad schematic (older format))
At the start: 53 parts, among them J1 Screw_Terminal_01x05, J2 Screw_Terminal_01x05, J3 Serial-Prog, J4 Conn_01x02, J5 NextionDisplay, J6 USB_B_Micro, J7 AUX, Q1 IRF3708, Q2 IRF3708, SW1 Flash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

Commit message: rotary Encoder added
Parts:
- C7, C9: footprint (none) -> Capacitor_SMD:C_1206_3216Metric_Pad1.42x1.75mm_HandSolder
- R11, R9: footprint (none) -> Resistor_SMD:R_1206_3216Metric_Pad1.42x1.75mm_HandSolder
- SW3: footprint (none) -> Rotary_Encoder:RotaryEncoder_Alps_EC12E-Switch_Vertical_H20mm
Changed lines of the file:
@@
 F 0 "SW3" H 2100 6300 50  0000 C CNN
 F 1 "Rotary_Encoder_Switch" H 2100 6050 50  0000 C CNN
-F 2 "" H 1950 6760 50  0001 C CNN
+F 2 "Rotary_Encoder:RotaryEncoder_Alps_EC12E-Switch_Vertical_H20mm" H 1950 6760 50  0001 C CNN
 F 3 "~" H 2100 6860 50  0001 C CNN
 	1    2100 6600
@@
 F 0 "R9" H 1050 6350 50  0000 L CNN
 F 1 "10K" H 1000 6250 50  0000 L CNN
-F 2 "" V 1130 6300 50  0001 C CNN
+F 2 "Resistor_SMD:R_1206_3216Metric_Pad1.42x1.75mm_HandSolder" V 1130 6300 50  0001 C CNN
 F 3 "~" H 1200 6300 50  0001 C CNN
 	1    1200 6300
@@
 F 0 "R11" H 1400 6650 50  0000 L CNN
 F 1 "10K" H 1400 6550 50  0000 L CNN
-F 2 "" V 1380 6300 50  0001 C CNN
+F 2 "Resistor_SMD:R_1206_3216Metric_Pad1.42x1.75mm_HandSolder" V 1380 6300 50  0001 C CNN
 F 3 "~" H 1450 6300 50  0001 C CNN
 	1    1450 6300
@@
 F 0 "C9" H 1500 7000 50  0000 L CNN
 F 1 "1u" H 1500 6800 50  0000 L CNN
-F 2 "" H 1488 6750 50  0001 C CNN
+F 2 "Capacitor_SMD:C_1206_3216Metric_Pad1.42x1.75mm_HandSolder" H 1488 6750 50  0001 C CNN
 F 3 "~" H 1450 6900 50  0001 C CNN
 	1    1450 6900
@@
 F 0 "C7" H 1000 7000 50  0000 L CNN
 F 1 "1u" H 1000 6800 50  0000 L CNN
-F 2 "" H 1238 6750 50  0001 C CNN
+F 2 "Capacitor_SMD:C_1206_3216Metric_Pad1.42x1.75mm_HandSolder" H 1238 6750 50  0001 C CNN
 F 3 "~" H 1200 6900 50  0001 C CNN
 	1    1200 6900

Commit message: ESP32 footprint added
Parts:
- U2: footprint module:ESP-WROOM-32-short -> RF_Module:ESP32-WROOM-32
Changed lines of the file:
@@
 F 0 "U2" H 2500 6400 60  0000 C CNN
 F 1 "ESP-WROOM-32" H 3125 6431 60  0000 C CNN
-F 2 "module:ESP-WROOM-32-short" H 3600 4900 60  0001 C CNN
+F 2 "RF_Module:ESP32-WROOM-32" H 3600 4900 60  0001 C CNN
 F 3 "" H 3600 4900 60  0001 C CNN
 	1    3150 5200

Commit message: rotary
Parts:
- SW3: footprint Rotary_Encoder:RotaryEncoder_Alps_EC12E-Switch_Vertical_H20mm -> Rotary_Encoder:RotaryEncoder_Alps_EC11E-Switch_Vertical_H20mm
- U2: footprint RF_Module:ESP32-WROOM-32 -> ESP32-footprints:ESP32-WROOM
Changed lines of the file:
@@
 F 0 "U2" H 2500 6400 60  0000 C CNN
 F 1 "ESP-WROOM-32" H 3125 6431 60  0000 C CNN
-F 2 "RF_Module:ESP32-WROOM-32" H 3600 4900 60  0001 C CNN
+F 2 "ESP32-footprints:ESP32-WROOM" H 3600 4900 60  0001 C CNN
 F 3 "" H 3600 4900 60  0001 C CNN
 	1    3150 5200
@@
 F 0 "SW3" H 2100 6300 50  0000 C CNN
 F 1 "Rotary_Encoder_Switch" H 2100 6050 50  0000 C CNN
-F 2 "Rotary_Encoder:RotaryEncoder_Alps_EC12E-Switch_Vertical_H20mm" H 1950 6760 50  0001 C CNN
+F 2 "Rotary_Encoder:RotaryEncoder_Alps_EC11E-Switch_Vertical_H20mm" H 1950 6760 50  0001 C CNN
 F 3 "~" H 2100 6860 50  0001 C CNN
 	1    2100 6600

Commit message: layout1
Parts:
- added TP8: Reserve-2, TestPoint:TestPoint_Pad_D1.5mm, symbol ESP32-wroom:Test_Point-Connector
- added TP9: Reserve-1, TestPoint:TestPoint_Pad_D1.5mm, symbol ESP32-wroom:Test_Point-Connector
- J1: value Screw_Terminal_01x05 -> Power
- J2: value Screw_Terminal_01x05 -> LED-out
- U1: value TLV70233_SOT23-5 -> TLV70233
Connections:
- net at J2.5 (Pin_5): now also TP9.1
- net at J2.6 (Pin_6): now also TP8.1
- no-connect marks 29 -> 27
Changed lines of the file:
@@
 P 2550 1450
 F 0 "U1" H 2550 1792 50  0000 C CNN
-F 1 "TLV70233_SOT23-5" H 2550 1701 50  0000 C CNN
+F 1 "TLV70233" H 2550 1701 50  0000 C CNN
 F 2 "Package_TO_SOT_SMD:SOT-23-5" H 2550 1775 50  0001 C CIN
 F 3 "http://www.ti.com/lit/ds/symlink/tlv712.pdf" H 2550 1450 50  0001 C CNN
@@
 	1    5700 4250
 	0    1    1    0
-$EndComp
-$Comp
-L Connector:Screw_Terminal_01x06 J1
-U 1 1 5BEC5924
-P 1100 3150
-F 0 "J1" H 1020 2625 50  0000 C CNN
-F 1 "Screw_Terminal_01x05" H 1020 2716 50  0000 C CNN
-F 2 "Connector_Phoenix_MSTB:PhoenixContact_MSTBVA_2,5_6-G-5,08_1x06_P5.08mm_Vertical" H 1100 3150 50  0001 C CNN
-F 3 "~" H 1100 3150 50  0001 C CNN
-	1    1100 3150
-	-1   0    0    1
 $EndComp
 Wire Wire Line
@@
 Wire Wire Line
 	1300 2850 1550 2850
-Connection ~ 1300 2850
 Connection ~ 3150 3400
 $Comp
@@
 P 5000 1250
 F 0 "J2" H 4920 725 50  0000 C CNN
-F 1 "Screw_Terminal_01x05" H 4920 816 50  0000 C CNN
+F 1 "LED-out" H 4920 816 50  0000 C CNN
 F 2 "Connector_Phoenix_MSTB:PhoenixContact_MSTBVA_2,5_6-G-5,08_1x06_P5.08mm_Vertical" H 5000 1250 50  0001 C CNN
 F 3 "~" H 5000 1250 50  0001 C CNN
@@
 NoConn ~ 4400 6750
 NoConn ~ 4400 6850
-NoConn ~ 5200 1050
-NoConn ~ 5200 950
 Wire Wire Line
 	8250 3900 8750 3900
@@
 U 1 1 5BE7BE7C
 P 7200 1750
-F 0 "JP2" H 7200 1565 50  0000 C CNN
+F 0 "JP2" H 7300 1950 50  0000 C CNN
 F 1 "USB-GND" H 7300 1850 50  0000 C CNN
 F 2 "Connector_PinHeader_2.54mm:PinHeader_1x02_P2.54mm_Vertical" H 7200 1750 50  0001 C CNN
@@
 Wire Wire Line
 	1200 6100 1200 6150
+Connection ~ 1300 2850
+$Comp
+L Connector:Screw_Terminal_01x06 J1
+U 1 1 5BEC5924
+P 1100 3150
+F 0 "J1" H 1020 2625 50  0000 C CNN
+F 1 "Power" H 1020 2716 50  0000 C CNN
+F 2 "Connector_Phoenix_MSTB:PhoenixContact_MSTBVA_2,5_6-G-5,08_1x06_P5.08mm_Vertical" H 1100 3150 50  0001 C CNN
+F 3 "~" H 1100 3150 50  0001 C CNN
+	1    1100 3150
+	-1   0    0    1
+$EndComp
+Wire Wire Line
+	5200 1050 5350 1050
+Wire Wire Line
+	5200 950  5350 950
+$Comp
+L ESP32-wroom:Test_Point-Connector TP9
+U 1 1 5C0C035B
+P 5350 1050
+F 0 "TP9" V 5300 1250 50  0000 L CNN
+F 1 "Reserve-1" V 5300 1400 50  0000 L CNN
+F 2 "TestPoint:TestPoint_Pad_D1.5mm" H 5550 1050 50  0001 C CNN
+F 3 "~" H 5550 1050 50  0001 C CNN
+	1    5350 1050
+	0    1    1    0
+$EndComp
+$Comp
+L ESP32-wroom:Test_Point-Connector TP8
+U 1 1 5C0C0AF1
+P 5350 950
+F 0 "TP8" V 5300 1150 50  0000 L CNN
+F 1 "Reserve-2" V 5300 1300 50  0000 L CNN
+F 2 "TestPoint:TestPoint_Pad_D1.5mm" H 5550 950 50  0001 C CNN
+F 3 "~" H 5550 950 50  0001 C CNN
+	1    5350 950
+	0    1    1    0
+$EndComp
 $EndSCHEMATC

Commit message: layout2
Parts:
- J3: value Serial-Prog -> Prog
- J4: value Conn_01x02 -> 3.3V
- SW3: value Rotary_Encoder_Switch -> Rotary_Encoder
- TP1: value Test_Point -> TP_3.3V
- TP7: value Test_Point -> TP_5V
Changed lines of the file:
@@
 U 1 1 5B370F86
 P 4400 3200
-F 0 "J3" H 4400 3500 50  0000 R CNN
-F 1 "Serial-Prog" H 4600 3600 50  0000 R CNN
+F 0 "J3" H 4550 3500 50  0000 R CNN
+F 1 "Prog" H 4550 2950 50  0000 R CNN
 F 2 "Connector_PinHeader_2.54mm:PinHeader_1x05_P2.54mm_Vertical" H 4400 3200 50  0001 C CNN
 F 3 "~" H 4400 3200 50  0001 C CNN
@@
 P 3850 1350
 F 0 "TP1" H 3908 1470 50  0000 L CNN
-F 1 "Test_Point" H 3908 1379 50  0000 L CNN
+F 1 "TP_3.3V" H 3908 1379 50  0000 L CNN
 F 2 "TestPoint:TestPoint_Pad_D1.5mm" H 4050 1350 50  0001 C CNN
 F 3 "~" H 4050 1350 50  0001 C CNN
@@
 P 1100 1350
 F 0 "TP7" H 1158 1470 50  0000 L CNN
-F 1 "Test_Point" H 900 1600 50  0000 L CNN
+F 1 "TP_5V" H 900 1600 50  0000 L CNN
 F 2 "TestPoint:TestPoint_Pad_D1.5mm" H 1300 1350 50  0001 C CNN
 F 3 "~" H 1300 1350 50  0001 C CNN
@@
 P 4050 1650
 F 0 "J4" H 4130 1642 50  0000 L CNN
-F 1 "Conn_01x02" H 3900 1400 50  0000 L CNN
+F 1 "3.3V" H 3900 1400 50  0000 L CNN
 F 2 "Connector_PinHeader_2.54mm:PinHeader_1x02_P2.54mm_Vertical" H 4050 1650 50  0001 C CNN
 F 3 "~" H 4050 1650 50  0001 C CNN
@@
 P 2100 6600
 F 0 "SW3" H 2100 6300 50  0000 C CNN
-F 1 "Rotary_Encoder_Switch" H 2100 6050 50  0000 C CNN
+F 1 "Rotary_Encoder" H 2100 6050 50  0000 C CNN
 F 2 "Rotary_Encoder:RotaryEncoder_Alps_EC11E-Switch_Vertical_H20mm" H 1950 6760 50  0001 C CNN
 F 3 "~" H 2100 6860 50  0001 C CNN

Commit message: Layouting3
Parts:
- added TP10: +12V, TestPoint:TestPoint_Pad_D1.5mm, symbol ESP32-wroom:Test_Point-Connector
- TP1: value TP_3.3V -> +3.3V
- TP3: value TP_Boot -> Boot
- TP4: value TP_Reset -> Reset
- TP7: value TP_5V -> +5V
Connections:
- net +12V: now also TP10.1
Changed lines of the file:
@@
 P 3750 3100
 F 0 "TP4" H 3550 3200 50  0000 L CNN
-F 1 "TP_Reset" H 3600 3350 50  0000 L CNN
+F 1 "Reset" H 3600 3350 50  0000 L CNN
 F 2 "TestPoint:TestPoint_Pad_D1.5mm" H 3950 3100 50  0001 C CNN
 F 3 "~" H 3950 3100 50  0001 C CNN
@@
 P 3750 3400
 F 0 "TP3" H 3550 3500 50  0000 L CNN
-F 1 "TP_Boot" H 3650 3300 50  0000 L CNN
+F 1 "Boot" H 3650 3300 50  0000 L CNN
 F 2 "TestPoint:TestPoint_Pad_D1.5mm" H 3950 3400 50  0001 C CNN
 F 3 "~" H 3950 3400 50  0001 C CNN
@@
 P 3850 1350
 F 0 "TP1" H 3908 1470 50  0000 L CNN
-F 1 "TP_3.3V" H 3908 1379 50  0000 L CNN
+F 1 "+3.3V" H 3908 1379 50  0000 L CNN
 F 2 "TestPoint:TestPoint_Pad_D1.5mm" H 4050 1350 50  0001 C CNN
 F 3 "~" H 4050 1350 50  0001 C CNN
@@
 P 1100 1350
 F 0 "TP7" H 1158 1470 50  0000 L CNN
-F 1 "TP_5V" H 900 1600 50  0000 L CNN
+F 1 "+5V" H 1050 1600 50  0000 L CNN
 F 2 "TestPoint:TestPoint_Pad_D1.5mm" H 1300 1350 50  0001 C CNN
 F 3 "~" H 1300 1350 50  0001 C CNN
@@
 	6200 3450 6600 3450
 Wire Wire Line
-	5400 3450 6200 3450
+	5400 3450 5700 3450
 Wire Wire Line
 	5200 1450 5350 1450
@@
 	0    1    1    0
 $EndComp
+$Comp
+L ESP32-wroom:Test_Point-Connector TP10
+U 1 1 5BF05B0B
+P 5700 3450
+F 0 "TP10" H 5500 3550 50  0000 L CNN
+F 1 "+12V" H 5550 3700 50  0000 L CNN
+F 2 "TestPoint:TestPoint_Pad_D1.5mm" H 5900 3450 50  0001 C CNN
+F 3 "~" H 5900 3450 50  0001 C CNN
+	1    5700 3450
+	1    0    0    -1
+$EndComp
+Connection ~ 5700 3450
+Wire Wire Line
+	5700 3450 6200 3450
 $EndSCHEMATC

Commit message: Layouting4
Parts:
- added TP11: Neo_unten, TestPoint:TestPoint_Pad_D1.5mm, symbol ESP32-wroom:Test_Point-Connector
- added TP12: Neo_oben, TestPoint:TestPoint_Pad_D1.5mm, symbol ESP32-wroom:Test_Point-Connector
- TP8: value Reserve-2 -> Res-2
- TP9: value Reserve-1 -> Res-1
Connections:
- net Neopixel_oben: now also TP12.1
- net Neopixel_unten: now also TP11.1
Changed lines of the file:
@@
 $EndComp
-Wire Wire Line
-	5400 6550 5700 6550
 Wire Wire Line
 	4800 7200 5500 7200
@@
 P 5350 1050
 F 0 "TP9" V 5300 1250 50  0000 L CNN
-F 1 "Reserve-1" V 5300 1400 50  0000 L CNN
+F 1 "Res-1" V 5300 1400 50  0000 L CNN
 F 2 "TestPoint:TestPoint_Pad_D1.5mm" H 5550 1050 50  0001 C CNN
 F 3 "~" H 5550 1050 50  0001 C CNN
@@
 P 5350 950
 F 0 "TP8" V 5300 1150 50  0000 L CNN
-F 1 "Reserve-2" V 5300 1300 50  0000 L CNN
+F 1 "Res-2" V 5300 1300 50  0000 L CNN
 F 2 "TestPoint:TestPoint_Pad_D1.5mm" H 5550 950 50  0001 C CNN
 F 3 "~" H 5550 950 50  0001 C CNN
@@
 Wire Wire Line
 	5700 3450 6200 3450
+$Comp
+L ESP32-wroom:Test_Point-Connector TP12
+U 1 1 5BF0810E
+P 5700 6500
+F 0 "TP12" H 5750 6650 50  0000 L CNN
+F 1 "Neo_oben" H 5550 6750 50  0000 L CNN
+F 2 "TestPoint:TestPoint_Pad_D1.5mm" H 5900 6500 50  0001 C CNN
+F 3 "~" H 5900 6500 50  0001 C CNN
+	1    5700 6500
+	1    0    0    -1
+$EndComp
+$Comp
+L ESP32-wroom:Test_Point-Connector TP11
+U 1 1 5BF083A5
+P 5500 6500
+F 0 "TP11" H 5300 6600 50  0000 L CNN
+F 1 "Neo_unten" H 5350 6750 50  0000 L CNN
+F 2 "TestPoint:TestPoint_Pad_D1.5mm" H 5700 6500 50  0001 C CNN
+F 3 "~" H 5700 6500 50  0001 C CNN
+	1    5500 6500
+	1    0    0    -1
+$EndComp
+Wire Wire Line
+	5400 6550 5700 6550
+Wire Wire Line
+	5700 6500 5700 6550
+Wire Wire Line
+	5500 6500 5500 6650
 $EndSCHEMATC

Commit message: gerberplot
Other:
- note added: "Rotary Encoder"
- moved on the sheet: C7, C9, R11, R9, SW3
Changed lines of the file:
@@
 Sheet 1 1
 Title "ESP32-wood-beam-lamp"
-Date ""
+Date "2018-11-18"
 Rev "1.0"
 Comp "Viktor Rees"
@@
 NoConn ~ 9100 4300
 NoConn ~ 150  3200
-$Comp
-L Device:Rotary_Encoder_Switch SW3
-U 1 1 5BEB6E38
-P 2100 6600
-F 0 "SW3" H 2100 6300 50  0000 C CNN
-F 1 "Rotary_Encoder" H 2100 6050 50  0000 C CNN
-F 2 "Rotary_Encoder:RotaryEncoder_Alps_EC11E-Switch_Vertical_H20mm" H 1950 6760 50  0001 C CNN
-F 3 "~" H 2100 6860 50  0001 C CNN
-	1    2100 6600
-	1    0    0    -1
-$EndComp
 Text Label 1950 5500 0    50   ~ 0
 ROT_A
@@
 L Device:R R9
 U 1 1 5BEF62E4
-P 1200 6300
-F 0 "R9" H 1050 6350 50  0000 L CNN
-F 1 "10K" H 1000 6250 50  0000 L CNN
-F 2 "Resistor_SMD:R_1206_3216Metric_Pad1.42x1.75mm_HandSolder" V 1130 6300 50  0001 C CNN
-F 3 "~" H 1200 6300 50  0001 C CNN
-	1    1200 6300
+P 1200 6650
+F 0 "R9" H 1050 6700 50  0000 L CNN
+F 1 "10K" H 1000 6600 50  0000 L CNN
+F 2 "Resistor_SMD:R_1206_3216Metric_Pad1.42x1.75mm_HandSolder" V 1130 6650 50  0001 C CNN
+F 3 "~" H 1200 6650 50  0001 C CNN
+	1    1200 6650
 	1    0    0    -1
 $EndComp
@@
 L Device:R R11
 U 1 1 5BF1348A
-P 1450 6300
-F 0 "R11" H 1400 6650 50  0000 L CNN
-F 1 "10K" H 1400 6550 50  0000 L CNN
-F 2 "Resistor_SMD:R_1206_3216Metric_Pad1.42x1.75mm_HandSolder" V 1380 6300 50  0001 C CNN
-F 3 "~" H 1450 6300 50  0001 C CNN
-	1    1450 6300
-	1    0    0    -1
-$EndComp
-Wire Wire Line
-	1450 7100 1450 7050
+P 1450 6650
+F 0 "R11" H 1400 7000 50  0000 L CNN
+F 1 "10K" H 1400 6900 50  0000 L CNN
+F 2 "Resistor_SMD:R_1206_3216Metric_Pad1.42x1.75mm_HandSolder" V 1380 6650 50  0001 C CNN
+F 3 "~" H 1450 6650 50  0001 C CNN
+	1    1450 6650
+	1    0    0    -1
+$EndComp
+Wire Wire Line
+	1450 7450 1450 7400
 $Comp
 L Device:C C9
 U 1 1 5BF22FF7
-P 1450 6900
-F 0 "C9" H 1500 7000 50  0000 L CNN
-F 1 "1u" H 1500 6800 50  0000 L CNN
-F 2 "Capacitor_SMD:C_1206_3216Metric_Pad1.42x1.75mm_HandSolder" H 1488 6750 50  0001 C CNN
-F 3 "~" H 1450 6900 50  0001 C CNN
-	1    1450 6900
-	1    0    0    -1
-$EndComp
-Connection ~ 1450 7050
+P 1450 7250
+F 0 "C9" H 1500 7350 50  0000 L CNN
+F 1 "1u" H 1500 7150 50  0000 L CNN
+F 2 "Capacitor_SMD:C_1206_3216Metric_Pad1.42x1.75mm_HandSolder" H 1488 7100 50  0001 C CNN
+F 3 "~" H 1450 7250 50  0001 C CNN
+	1    1450 7250
+	1    0    0    -1
+$EndComp
+Connection ~ 1450 7400
 $Comp
 L power:GND #PWR026
 U 1 1 5BF13867
-P 1450 7100
-F 0 "#PWR026" H 1450 6850 50  0001 C CNN
-F 1 "GND" H 1455 6927 50  0000 C CNN
-F 2 "" H 1450 7100 50  0001 C CNN
-F 3 "" H 1450 7100 50  0001 C CNN
-	1    1450 7100
+P 1450 7450
+F 0 "#PWR026" H 1450 7200 50  0001 C CNN
+F 1 "GND" H 1455 7277 50  0000 C CNN
+F 2 "" H 1450 7450 50  0001 C CNN
+F 3 "" H 1450 7450 50  0001 C CNN
+	1    1450 7450
 	1    0    0    -1
 $EndComp
@@
 L Device:C C7
 U 1 1 5BF229E6
-P 1200 6900
-F 0 "C7" H 1000 7000 50  0000 L CNN
-F 1 "1u" H 1000 6800 50  0000 L CNN
-F 2 "Capacitor_SMD:C_1206_3216Metric_Pad1.42x1.75mm_HandSolder" H 1238 6750 50  0001 C CNN
-F 3 "~" H 1200 6900 50  0001 C CNN
-	1    1200 6900
-	1    0    0    -1
-$EndComp
-Wire Wire Line
-	1200 7050 1450 7050
-Wire Wire Line
-	1200 6450 1200 6500
-Wire Wire Line
-	1450 6450 1450 6700
-Wire Wire Line
-	1800 6500 1650 6500
-Connection ~ 1200 6500
-Wire Wire Line
-	1200 6500 1200 6750
-Wire Wire Line
-	1800 6700 1700 6700
-Connection ~ 1450 6700
-Wire Wire Line
-	1450 6700 1450 6750
+P 1200 7250
+F 0 "C7" H 1000 7350 50  0000 L CNN
+F 1 "1u" H 1000 7150 50  0000 L CNN
+F 2 "Capacitor_SMD:C_1206_3216Metric_Pad1.42x1.75mm_HandSolder" H 1238 7100 50  0001 C CNN
+F 3 "~" H 1200 7250 50  0001 C CNN
+	1    1200 7250
+	1    0    0    -1
+$EndComp
+Wire Wire Line
+	1200 7400 1450 7400
+Wire Wire Line
+	1200 6800 1200 6850
+Wire Wire Line
+	1450 6800 1450 7050
+Wire Wire Line
+	1800 6850 1700 6850
+Connection ~ 1200 6850
+Wire Wire Line
+	1200 6850 1200 7100
+Wire Wire Line
+	1800 7050 1750 7050
+Connection ~ 1450 7050
+Wire Wire Line
+	1450 7050 1450 7100
 Wire Wire Line
 	1950 5700 2200 5700
-Wire Wire Line
-	1450 7050 1800 7050
-Wire Wire Line
-	2450 7050 2450 6700
-Wire Wire Line
-	2450 6700 2400 6700
-Wire Wire Line
-	2400 6500 2450 6500
-Wire Wire Line
-	2450 6500 2450 6200
 Wire Wire Line
 	2450 6200 2200 6200
@@
 	2200 5700 2250 5700
 Wire Wire Line
-	1650 5500 1650 6500
-Wire Wire Line
-	1650 5500 2250 5500
-Wire Wire Line
-	1650 6500 1200 6500
-Wire Wire Line
-	1700 5600 1700 6700
-Wire Wire Line
-	1700 5600 2250 5600
-Connection ~ 1700 6700
-Wire Wire Line
-	1700 6700 1450 6700
-Connection ~ 1800 7050
-Wire Wire Line
-	1800 7050 2450 7050
-Connection ~ 1650 6500
-Wire Wire Line
-	1800 6600 1800 7050
+	1700 5500 1700 6850
+Wire Wire Line
+	1700 5500 2250 5500
+Wire Wire Line
+	1700 6850 1200 6850
+Wire Wire Line
+	1750 5600 1750 7050
+Wire Wire Line
+	1750 5600 2250 5600
+Connection ~ 1750 7050
+Wire Wire Line
+	1750 7050 1450 7050
+Connection ~ 1700 6850
 $Comp
 L power:+3.3V #PWR024
 U 1 1 5C08ACFD
-P 1200 6050
-F 0 "#PWR024" H 1200 5900 50  0001 C CNN
-F 1 "+3.3V" H 1215 6223 50  0000 C CNN
-F 2 "" H 1200 6050 50  0001 C CNN
-F 3 "" H 1200 6050 50  0001 C CNN
-	1    1200 6050
-	1    0    0    -1
-$EndComp
-Wire Wire Line
-	1200 6050 1200 6100
-Wire Wire Line
-	1450 6150 1450 6100
-Wire Wire Line
-	1450 6100 1200 6100
-Connection ~ 1200 6100
-Wire Wire Line
-	1200 6100 1200 6150
+P 1200 6400
+F 0 "#PWR024" H 1200 6250 50  0001 C CNN
+F 1 "+3.3V" H 1215 6573 50  0000 C CNN
+F 2 "" H 1200 6400 50  0001 C CNN
+F 3 "" H 1200 6400 50  0001 C CNN
+	1    1200 6400
+	1    0    0    -1
+$EndComp
+Wire Wire Line
+	1200 6400 1200 6450
+Wire Wire Line
+	1450 6500 1450 6450
+Wire Wire Line
+	1450 6450 1200 6450
+Connection ~ 1200 6450
+Wire Wire Line
+	1200 6450 1200 6500
 Connection ~ 1300 2850
 $Comp
@@
 Wire Wire Line
 	5500 6500 5500 6650
+$Comp
+L Device:Rotary_Encoder_Switch SW3
+U 1 1 5BEB6E38
+P 2100 6950
+F 0 "SW3" H 2100 6650 50  0000 C CNN
+F 1 "Rotary_Encoder" H 2100 7200 50  0000 C CNN
+F 2 "Rotary_Encoder:RotaryEncoder_Alps_EC11E-Switch_Vertical_H20mm" H 1950 7110 50  0001 C CNN
+F 3 "~" H 2100 7210 50  0001 C CNN
+	1    2100 6950
+	1    0    0    -1
+$EndComp
+Wire Wire Line
+	1450 7400 1650 7400
+Wire Wire Line
+	1800 6950 1650 6950
+Wire Wire Line
+	1650 6950 1650 7400
+Connection ~ 1650 7400
+Wire Wire Line
+	1650 7400 2450 7400
+Wire Wire Line
+	2400 6850 2450 6850
+Wire Wire Line
+	2450 6200 2450 6850
+Wire Wire Line
+	2400 7050 2450 7050
+Wire Wire Line
+	2450 7050 2450 7400
+Wire Notes Line
+	600  6100 2500 6100
+Wire Notes Line
+	2500 6100 2500 7700
+Wire Notes Line
+	2500 7700 600  7700
+Wire Notes Line
+	600  7700 600  6100
+Text Notes 650  6200 0    50   ~ 0
+Rotary Encoder
 $EndSCHEMATC
