File: kicad/ESP32-wood-beam-lamp.sch (KiCad schematic (older format))
At the start: 58 parts, among them J1 Power, J2 LED-out, J3 Prog, J4 3.3V, J5 NextionDisplay, J6 USB_B_Micro, J7 AUX, Q1 IRF3708, Q2 IRF3708, SW1 Flash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

Commit message: .
Parts:
- R11, R9: value 10K -> 10k
- R5, R6: value 100K -> 100k
Changed lines of the file:
@@
 P 5500 6850
 F 0 "R5" H 5450 6400 50  0000 L CNN
-F 1 "100K" H 5400 6300 50  0000 L CNN
+F 1 "100k" H 5400 6300 50  0000 L CNN
 F 2 "Resistor_SMD:R_1206_3216Metric_Pad1.42x1.75mm_HandSolder" V 5430 6850 50  0001 C CNN
 F 3 "~" H 5500 6850 50  0001 C CNN
@@
 P 5700 6850
 F 0 "R6" H 5650 6400 50  0000 L CNN
-F 1 "100K" H 5650 6300 50  0000 L CNN
+F 1 "100k" H 5650 6300 50  0000 L CNN
 F 2 "Resistor_SMD:R_1206_3216Metric_Pad1.42x1.75mm_HandSolder" V 5630 6850 50  0001 C CNN
 F 3 "~" H 5700 6850 50  0001 C CNN
@@
 P 1200 6650
 F 0 "R9" H 1050 6700 50  0000 L CNN
-F 1 "10K" H 1000 6600 50  0000 L CNN
+F 1 "10k" H 1000 6600 50  0000 L CNN
 F 2 "Resistor_SMD:R_1206_3216Metric_Pad1.42x1.75mm_HandSolder" V 1130 6650 50  0001 C CNN
 F 3 "~" H 1200 6650 50  0001 C CNN
@@
 P 1450 6650
 F 0 "R11" H 1400 7000 50  0000 L CNN
-F 1 "10K" H 1400 6900 50  0000 L CNN
+F 1 "10k" H 1400 6900 50  0000 L CNN
 F 2 "Resistor_SMD:R_1206_3216Metric_Pad1.42x1.75mm_HandSolder" V 1380 6650 50  0001 C CNN
 F 3 "~" H 1450 6650 50  0001 C CNN
