File: kicad/ESP32-wood-beam-lamp.kicad_pcb (KiCad board)
At the start: 2 copper layers, 53 parts, among them J1 Screw_Terminal_01x05, J2 Screw_Terminal_01x05, J3 Serial-Prog, J4 Conn_01x02, J5 NextionDisplay, J6 USB_B_Micro, J7 AUX, Q1 IRF3708, Q2 IRF3708, SW1 Flash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

Commit message: layout1
Parts:
- added ?: M3, MountingHole:MountingHole_3.2mm_M3, F.Cu at (96.0, 126.0)
- added ?: M3, MountingHole:MountingHole_3.2mm_M3, F.Cu at (44.0, 126.0)
- added ?: M3, MountingHole:MountingHole_3.2mm_M3, F.Cu at (44.0, 34.0)
- added ?: M3, MountingHole:MountingHole_3.2mm_M3, F.Cu at (96.0, 34.0)
- added TP8: Reserve-2, TestPoint:TestPoint_Pad_D1.5mm, F.Cu at (22.6, 54.9)
- added TP9: Reserve-1, TestPoint:TestPoint_Pad_D1.5mm, F.Cu at (25.2, 54.9)
- J1: value Screw_Terminal_01x05 -> Power
- J2: value Screw_Terminal_01x05 -> LED-out
- SW3: footprint Rotary_Encoder:RotaryEncoder_Alps_EC12E-Switch_Vertical_H20mm -> Rotary_Encoder:RotaryEncoder_Alps_EC11E-Switch_Vertical_H20mm
- U1: value TLV70233_SOT23-5 -> TLV70233
- moved C3 134.1 mm to (33.3, 98.3)
- moved C9 134.1 mm to (21.8, 107.8)
- moved D1 134.1 mm to (18.2, 119.3)
- moved R25 134.1 mm to (18.5, 110.1)
- moved R3 134.1 mm to (18.5, 112.4)
- moved R5 134.1 mm to (18.5, 114.7)
- moved TP2 134.1 mm to (37.1, 96.1)
- moved TP3 134.1 mm to (37.1, 98.7)
- moved TP7 134.1 mm to (22.2, 117.1)
- moved U1 134.1 mm to (27.9, 110.8)
- moved C2 134.1 mm to (23.5, 114.7)
- moved C7 134.1 mm to (33.3, 96.0)
- moved R10 134.1 mm to (18.4, 117.0)
- moved R11 134.1 mm to (31.7, 102.9)
- moved R12 134.1 mm to (23.5, 112.4)
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Routing:
- net +12V: track 0.00 -> 53.3 mm
- net GND: track 0.00 -> 33.4 mm
- net +5V: track 0.00 -> 20.1 mm
- net /LED_out2: track 0.00 -> 16.8 mm
- net /LED_out1: track 0.00 -> 15.8 mm
- net Net-(J6-Pad6): track 0.00 -> 12.9 mm
- net Net-(D5-Pad2): track 0.00 -> 3.56 mm
- net Net-(J6-Pad1): track 0.00 -> 3.41 mm
- net Net-(J6-Pad5): track 0.00 -> 3.20 mm
- net Net-(D4-Pad2): track 0.00 -> 3.06 mm
- added copper zone on B.Cu, net GND
Other:
- board outline added: 60 x 100 mm
- net class XL added: clearance 0.4, trace_width 0.5, via_dia 0.8, via_drill 0.4
- net class XXL added: clearance 0.4, trace_width 2, via_dia 0.8, via_drill 0.4

Commit message: layout2
Parts:
- added IN+: +12V, TestPoint:TestPoint_THTPad_2.5x2.5mm_Drill1.2mm, F.Cu at (59.3, 107.7)
- added IN-: GND, TestPoint:TestPoint_THTPad_2.5x2.5mm_Drill1.2mm, F.Cu at (77.0, 107.7)
- added OUT+: +5v, TestPoint:TestPoint_THTPad_2.5x2.5mm_Drill1.2mm, F.Cu at (59.3, 69.6)
- added OUT-: GND, TestPoint:TestPoint_THTPad_2.5x2.5mm_Drill1.2mm, F.Cu at (77.0, 69.6)
- J3: value Serial-Prog -> Prog
- J4: value Conn_01x02 -> 3.3V
- SW3: value Rotary_Encoder_Switch -> Rotary_Encoder
- TP1: value Test_Point -> +3.3V
- TP7: value Test_Point -> +5V
- moved R1 85.3 mm to (95.6, 39.3)
- moved J4 79.3 mm to (47.3, 110.5), turned to 90 degrees
- moved J3 79.2 mm to (86.7, 44.5), turned to 90 degrees
- moved R3 78.0 mm to (82.2, 67.4), turned to 270 degrees
- moved R6 77.8 mm to (83.4, 60.5)
- moved R5 75.9 mm to (82.2, 73.4), turned to 270 degrees
- moved R13 75.7 mm to (94.9, 83.6), turned to 270 degrees
- moved TP6 75.6 mm to (81.2, 102.6)
- moved TP9 75.5 mm to (97.1, 77.7)
- moved TP8 75.1 mm to (94.1, 77.8)
- moved J5 72.4 mm to (88.3, 56.4), turned to 180 degrees
- moved TP3 72.2 mm to (97.8, 59.6)
- moved TP4 71.2 mm to (59.3, 33.6)
- moved TP1 68.3 mm to (43.3, 110.7)
- moved C6 68.0 mm to (93.6, 59.0), turned to 180 degrees
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Routing:
- net GND: track 33.4 -> 145.0 mm
- net +5V: track 20.1 -> 105.6 mm
- net +3V3: track 0.00 -> 41.9 mm, vias 0 -> 1
- net +12V: track 53.3 -> 83.7 mm
- net Net-(Q1-Pad1): track 0.00 -> 26.2 mm
- net Net-(Q2-Pad1): track 0.00 -> 13.0 mm
- net /LED_out1: track 15.8 -> 23.0 mm
- net /LED_out2: track 16.8 -> 24.0 mm
- net Net-(D3-Pad1): track 0.00 -> 4.52 mm
Other:
- net class XL: clearance 0.4 -> 0.3

Commit message: Layouting3
Parts:
- added REF**: KiCad-Logo_12mm_SilkScreen, Symbol:KiCad-Logo_12mm_SilkScreen, B.Cu at (54.9, 52.3)
- added TP10: +12V, TestPoint:TestPoint_Pad_D1.5mm, F.Cu at (75.8, 114.1)
- TP3: value TP_Boot -> Boot
- TP4: value TP_Reset -> Reset
- moved J4 29.2 mm to (75.6, 118.1)
- moved TP4 26.1 mm to (85.3, 32.5)
- moved TP1 25.1 mm to (68.2, 114.1)
- moved C8 20.7 mm to (60.5, 61.4)
- moved TP9 18.5 mm to (81.3, 87.4)
- moved R6 16.8 mm to (81.8, 77.3), turned to 90 degrees
- moved TP8 13.6 mm to (81.3, 82.3)
- moved R4 7.06 mm to (80.8, 66.5)
- moved R3 3.64 mm to (80.8, 64.0), turned to 180 degrees
- moved R5 2.87 mm to (81.8, 70.6)
- moved TP7 1.85 mm to (72.0, 114.1)
- moved TP2 1.37 mm to (79.6, 114.1)
- moved C9 1.34 mm to (57.4, 61.2)
- moved R1 0.87 mm to (95.5, 40.1)
- moved R10 0.84 mm to (41.5, 61.2)
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Routing:
- net GND: track 145.0 -> 427.4 mm, vias 0 -> 7
- net +3V3: track 41.9 -> 258.7 mm, vias 1 -> 8
- net /SCL: track 0.00 -> 66.3 mm, vias 0 -> 3
- net /SDA: track 0.00 -> 63.1 mm, vias 0 -> 2
- net Net-(Q1-Pad1): track 26.2 -> 81.1 mm, vias 0 -> 2
- net Net-(Q2-Pad1): track 13.0 -> 65.8 mm, vias 0 -> 2
- net /EN: track 0.00 -> 49.8 mm, vias 0 -> 2
- net +5V: track 105.6 -> 150.3 mm, vias 0 -> 2
- net /Neopixel_unten: track 0.00 -> 40.0 mm, vias 0 -> 1
- net /Neopixel_oben: track 0.14 -> 36.3 mm, vias 0 -> 2
- net Net-(U2-Pad16): track 0.00 -> 35.9 mm, vias 0 -> 2
- net /ROT_SW: track 0.00 -> 33.9 mm
- net /BOOT: track 0.00 -> 32.3 mm
- net +12V: track 83.7 -> 114.4 mm, vias 0 -> 5
- net Net-(U2-Pad23): track 0.00 -> 29.6 mm, vias 0 -> 2
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- added copper zone on F.Cu, net GND
Other:
- board text added: "ESP32-wood-beam-lamp R1.0 2018.11.17"

Commit message: Layouting4
Parts:
- added TP11: Neo_unten, TestPoint:TestPoint_Pad_D1.5mm, F.Cu at (81.3, 97.5)
- added TP12: Neo_oben, TestPoint:TestPoint_Pad_D1.5mm, F.Cu at (81.3, 92.5)
- TP8: value Reserve-2 -> Res-2
- TP9: value Reserve-1 -> Res-1
Routing:
- net /Neopixel_unten: track 40.0 -> 47.1 mm
- net /Neopixel_oben: track 36.3 -> 43.4 mm
Other:
- board text added: "ESP32-wood-beam-lamp R1.0"
- board text added: "Viktor Rees 2018.11.17"
- board text removed: "ESP32-wood-beam-lamp R1.0 2018.11.17"
Changed lines of the file:
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@@
   (general
     (thickness 1.6)
-    (drawings 12)
-    (tracks 548)
+    (drawings 13)
+    (tracks 550)
     (zones 0)
-    (modules 65)
+    (modules 67)
     (nets 64)
   )
   (page A4)
   (layers
-    (0 F.Cu signal)
-    (31 B.Cu signal)
+    (0 F.Cu signal hide)
+    (31 B.Cu signal hide)
     (32 B.Adhes user hide)
     (33 F.Adhes user hide)
@@
     (46 B.CrtYd user)
     (47 F.CrtYd user)
-    (48 B.Fab user)
+    (48 B.Fab user hide)
     (49 F.Fab user hide)
   )
@@
     (tags "resistor handsolder")
     (attr smd)
-    (fp_text reference R6 (at -1.016 -2.032 90) (layer F.SilkS)
+    (fp_text reference R6 (at 0.0365 -1.524 90) (layer F.SilkS)
       (effects (font (size 1 1) (thickness 0.15)))
     )
@@
     (tags "resistor handsolder")
     (attr smd)
-    (fp_text reference R3 (at -3.4782 0.1778 180) (layer F.SilkS)
+    (fp_text reference R3 (at 3.556 0.508 180) (layer F.SilkS)
       (effects (font (size 1 1) (thickness 0.15)))
     )
@@
     (tags "resistor handsolder")
     (attr smd)
-    (fp_text reference R4 (at 3.5417 -0.0635) (layer F.SilkS)
+    (fp_text reference R4 (at -4.1005 0.508) (layer F.SilkS)
       (effects (font (size 1 1) (thickness 0.15)))
     )
@@
     (tags "test point SMD pad")
     (attr virtual)
-    (fp_text reference TP8 (at -2.9464 -0.6096) (layer F.SilkS)
+    (fp_text reference TP8 (at 0 -1.524) (layer F.SilkS)
       (effects (font (size 1 1) (thickness 0.15)))
     )
-    (fp_text value Reserve-2 (at 0 1.75) (layer F.Fab)
+    (fp_text value Res-2 (at 0 1.75) (layer F.SilkS)
       (effects (font (size 1 1) (thickness 0.15)))
     )
@@
     (tags "test point SMD pad")
     (attr virtual)
-    (fp_text reference TP9 (at 1.1176 -1.5367) (layer F.SilkS)
+    (fp_text reference TP9 (at 0 -1.5367) (layer F.SilkS)
       (effects (font (size 1 1) (thickness 0.15)))
     )
-    (fp_text value Reserve-1 (at 0 1.75) (layer F.Fab)
+    (fp_text value Res-1 (at 0 1.75) (layer F.SilkS)
       (effects (font (size 1 1) (thickness 0.15)))
     )
@@
       (xy -12.322794 5.02551) (xy -11.847446 5.025459)) (layer B.SilkS) (width 0.01))
   )
-  (gr_text "ESP32-wood-beam-lamp R1.0 2018.11.17" (at 44.196 95.504 90) (layer B.SilkS)
+  (module TestPoint:TestPoint_Pad_D1.5mm (layer F.Cu)
+    (at 81.28 97.536)
+    (descr "SMD pad as test Point, diameter 1.5mm")
+    (tags "test point SMD pad")
+    (attr virtual)
+    (fp_text reference TP11 (at 0 -1.648) (layer F.SilkS)
+      (effects (font (size 1 1) (thickness 0.15)))
+    )
+    (fp_text value Neo_unten (at -2.032 1.75) (layer F.SilkS)
+      (effects (font (size 1 1) (thickness 0.15)))
+    )
+    (fp_text user %R (at 0 -1.65) (layer F.Fab)
+      (effects (font (size 1 1) (thickness 0.15)))
+    )
+    (fp_circle (center 0 0) (end 1.25 0) (layer F.CrtYd) (width 0.05))
+    (fp_circle (center 0 0) (end 0 0.95) (layer F.SilkS) (width 0.12))
+    (pad 1 smd circle (at 0 0) (size 1.5 1.5) (layers F.Cu F.Mask)
+      (net 12 /Neopixel_unten))
+  )
+  (module TestPoint:TestPoint_Pad_D1.5mm (layer F.Cu)
+    (at 81.28 92.456)
+    (descr "SMD pad as test Point, diameter 1.5mm")
+    (tags "test point SMD pad")
+    (attr virtual)
+    (fp_text reference TP12 (at 0 -1.648) (layer F.SilkS)
+      (effects (font (size 1 1) (thickness 0.15)))
+    )
+    (fp_text value Neo_oben (at -1.524 1.75) (layer F.SilkS)
+      (effects (font (size 1 1) (thickness 0.15)))
+    )
+    (fp_circle (center 0 0) (end 0 0.95) (layer F.SilkS) (width 0.12))
+    (fp_circle (center 0 0) (end 1.25 0) (layer F.CrtYd) (width 0.05))
+    (fp_text user %R (at 0 -1.65) (layer F.Fab)
+      (effects (font (size 1 1) (thickness 0.15)))
+    )
+    (pad 1 smd circle (at 0 0) (size 1.5 1.5) (layers F.Cu F.Mask)
+      (net 13 /Neopixel_oben))
+  )
+  (gr_text "Viktor Rees 2018.11.17" (at 45.72 91.44 90) (layer B.SilkS)
+    (effects (font (size 1.5 1.5) (thickness 0.3)) (justify mirror))
+  )
+  (gr_text "ESP32-wood-beam-lamp R1.0 " (at 42.164 96.52 90) (layer B.SilkS)
     (effects (font (size 1.5 1.5) (thickness 0.3)) (justify mirror))
   )
@@
   (segment (start 80.2275 69.1245) (end 79.756 69.596) (width 0.25) (layer F.Cu) (net 12))
   (segment (start 81.788 69.1245) (end 80.2275 69.1245) (width 0.25) (layer F.Cu) (net 12))
+  (segment (start 81.28 97.536) (end 88.392 97.536) (width 0.25) (layer F.Cu) (net 12))
   (segment (start 88.2904 92.5576) (end 88.392 92.456) (width 0.25) (layer F.Cu) (net 13))
   (segment (start 84.18089 86.95489) (end 84.18089 79.248) (width 0.25) (layer B.Cu) (net 13))
@@
   (segment (start 83.67289 78.74) (end 84.18089 79.248) (width 0.25) (layer F.Cu) (net 13))
   (segment (start 81.788 78.74) (end 83.67289 78.74) (width 0.25) (layer F.Cu) (net 13))
+  (segment (start 81.28 92.456) (end 88.392 92.456) (width 0.25) (layer F.Cu) (net 13))
   (segment (start 81.28 87.376) (end 88.392 87.376) (width 0.25) (layer F.Cu) (net 14))
   (segment (start 81.28 82.296) (end 88.392 82.296) (width 0.25) (layer F.Cu) (net 15))

Commit message: gerberplot
Parts:
- added ?: PinHeader_1x10_P2.54mm_Vertical, Connector_PinHeader_2.54mm:PinHeader_1x10_P2.54mm_Vertical, F.Cu at (55.9, 73.7)
- added ?: PinHeader_1x10_P2.54mm_Vertical, Connector_PinHeader_2.54mm:PinHeader_1x10_P2.54mm_Vertical, F.Cu at (43.2, 73.7)
- added ?: PinHeader_1x10_P2.54mm_Vertical, Connector_PinHeader_2.54mm:PinHeader_1x10_P2.54mm_Vertical, F.Cu at (45.7, 73.7)
- added ?: PinHeader_1x10_P2.54mm_Vertical, Connector_PinHeader_2.54mm:PinHeader_1x10_P2.54mm_Vertical, F.Cu at (48.3, 73.7)
- added ?: PinHeader_1x10_P2.54mm_Vertical, Connector_PinHeader_2.54mm:PinHeader_1x10_P2.54mm_Vertical, F.Cu at (50.8, 73.7)
- added ?: PinHeader_1x10_P2.54mm_Vertical, Connector_PinHeader_2.54mm:PinHeader_1x10_P2.54mm_Vertical, F.Cu at (53.3, 73.7)
- added REF**: Symbol_GNU-Logo_SilkscreenTop, Symbol:Symbol_GNU-Logo_SilkscreenTop, B.Cu at (69.6, 48.3)
- added REF**: OSHW-Logo2_14.6x12mm_SilkScreen, Symbol:OSHW-Logo2_14.6x12mm_SilkScreen, B.Cu at (49.3, 108.7)
- REF**: moved to F.Cu
- moved REF** 39.2 mm to (67.6, 89.4), turned to 90 degrees
Routing:
- net +3V3: track 258.7 -> 266.6 mm
- net /SCL: track 66.3 -> 73.5 mm
- net /SDA: track 63.1 -> 70.2 mm
- net +5V: track 150.3 -> 156.2 mm
- net GND: track 427.4 -> 430.2 mm
Other:
- board text added: "woodbeamlamp ESP32 R1.0 Viktor Rees"
